File: Voyager87.kicad_pcb (KiCad board)
At the start: 2 copper layers, 343.7 x 123.4 mm, 305 parts, among them J1 AVR-ISP-6, Q1 DSS60601MZ4-13, SW1 SW_Push, U1 AT90USB1286-AU, U2 PRTR5V0U2X, Y1 16MHz

Commit message: Progress
Parts:
- C5: value 10uF -> 1uF
- MX_LALT2: footprint MX_Alps_Hybrid:MX-1.5U -> MX_Alps_Hybrid:MX-1.5U-FLIPPED
- MX_LGUI2: footprint MX_Alps_Hybrid:MX-1U -> MX_Alps_Hybrid:MX-1U-FLIPPED
- MX_RALT2: footprint MX_Alps_Hybrid:MX-1.5U-FLIPPED -> MX_Alps_Hybrid:MX-1.5U
- MX_RCTRL1, MX_RGUI1, MX_RMENU1: footprint MX_Alps_Hybrid:MX-1.25U -> MX_Alps_Hybrid:MX-1.25U-FLIPPED
- moved D52 534.2 mm to (62.7, 100.0), turned to 90 degrees
- moved R1 494.4 mm to (55.6, 43.7), turned to 90 degrees
- moved R3 492.2 mm to (112.7, 43.7), turned to 90 degrees
- moved R20 489.1 mm to (112.7, 67.5), turned to 90 degrees
- moved R17 488.7 mm to (55.6, 67.5), turned to 90 degrees
- moved D37 486.7 mm to (103.2, 81.0), turned to 90 degrees
- moved R35 486.5 mm to (60.3, 86.5), turned to 90 degrees
- moved D54 480.2 mm to (108.0, 100.0), turned to 90 degrees
- moved D39 477.1 mm to (141.3, 81.0), turned to 90 degrees
- moved R14 475.8 mm to (79.4, 124.6), turned to 90 degrees
- moved R18 467.0 mm to (74.6, 67.5), turned to 90 degrees
- moved R2 466.6 mm to (93.7, 43.7), turned to 90 degrees
- moved R19 458.9 mm to (93.7, 67.5), turned to 90 degrees
- moved D55 456.8 mm to (127.0, 100.0), turned to 90 degrees
- moved D1 452.1 mm to (55.6, 38.1), turned to 90 degrees
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Connections:
- MX_LALT2 pad 1: Net-(MX_LALT2-Pad1) -> COL2
- MX_LALT2 pad 2: Net-(MX_LALT2-Pad2) -> Net-(D86-Pad2)
- MX_LALT2 pad 3: Net-(MX_LALT2-Pad3) -> +5V
- MX_LALT2 pad 4: Net-(MX_LALT2-Pad4) -> Net-(MX_LALT1-Pad4)
- MX_LGUI2 pad 1: Net-(D85-Pad2) -> COL1
- MX_LGUI2 pad 2: COL1 -> Net-(D85-Pad2)
- MX_LSHIFT2 pad 1: Net-(MX_LSHIFT2-Pad1) -> COL0
- MX_LSHIFT2 pad 2: Net-(MX_LSHIFT2-Pad2) -> Net-(D67-Pad2)
- MX_LSHIFT2 pad 3: Net-(MX_LSHIFT2-Pad3) -> +5V
- MX_LSHIFT2 pad 4: Net-(MX_LSHIFT2-Pad4) -> Net-(MX_LSHIFT1-Pad4)
- MX_RALT2 pad 1: Net-(D91-Pad2) -> COL11
- MX_RALT2 pad 2: COL11 -> Net-(D91-Pad2)
- MX_RCTRL2 pad 1: Net-(MX_RCTRL2-Pad1) -> COL13
- MX_RCTRL2 pad 2: Net-(MX_RCTRL2-Pad2) -> Net-(D82-Pad2)
- MX_RCTRL2 pad 3: Net-(MX_RCTRL2-Pad3) -> +5V
- MX_RCTRL2 pad 4: Net-(MX_RCTRL2-Pad4) -> Net-(MX_RCTRL1-Pad4)
- MX_RETURN2 pad 1: Net-(MX_RETURN2-Pad1) -> COL13
- MX_RETURN2 pad 2: Net-(MX_RETURN2-Pad2) -> Net-(D65-Pad2)
- MX_RETURN2 pad 3: Net-(MX_RETURN2-Pad3) -> +5V
- MX_RETURN2 pad 4: Net-(MX_RETURN2-Pad4) -> Net-(MX_RETURN1-Pad4)
- MX_RGUI2 pad 1: Net-(MX_RGUI2-Pad1) -> COL12
- MX_RGUI2 pad 2: Net-(MX_RGUI2-Pad2) -> Net-(D81-Pad2)
- MX_RGUI2 pad 3: Net-(MX_RGUI2-Pad3) -> +5V
- MX_RMENU1 pad 4: Net-(MX_RMENU1-Pad4) -> Net-(MX_RGUI2-Pad4)
- MX_RSHIFT2 pad 1: Net-(MX_RSHIFT2-Pad1) -> COL12
- MX_RSHIFT2 pad 2: Net-(MX_RSHIFT2-Pad2) -> Net-(D78-Pad2)
- MX_RSHIFT2 pad 3: Net-(MX_RSHIFT2-Pad3) -> +5V
- MX_RSHIFT2 pad 4: Net-(MX_RSHIFT2-Pad4) -> Net-(MX_RSHIFT1-Pad4)
- MX_SP2 pad 1: Net-(D87-Pad2) -> COL6
- MX_SP2 pad 2: COL6 -> Net-(D87-Pad2)
- MX_\2 pad 1: Net-(MX_\2-Pad1) -> COL13
- MX_\2 pad 2: Net-(MX_\2-Pad2) -> Net-(D48-Pad2)
- MX_\2 pad 3: Net-(MX_\2-Pad3) -> +5V
- MX_\2 pad 4: Net-(MX_\2-Pad4) -> Net-(MX_\1-Pad4)
- R81 pad 1: Net-(MX_RMENU1-Pad4) -> Net-(MX_RGUI2-Pad4)
- U1 pad 31: Net-(U1-Pad31) -> COL16
- U1 pad 32: ROW0 -> COL15
- U1 pad 35: COL16 -> Net-(U1-Pad35)
- U1 pad 36: COL15 -> Net-(U1-Pad36)
- U1 pad 37: Net-(U1-Pad37) -> ROW0
Routing:
- net +5V: track 0.00 -> 1138.9 mm, vias 0 -> 8
- net COL6: track 0.00 -> 708.8 mm
- net COL7: track 0.00 -> 690.8 mm
- net COL5: track 0.00 -> 621.4 mm
- net COL8: track 0.00 -> 574.4 mm
- net COL4: track 0.00 -> 564.4 mm, vias 0 -> 1
- net COL3: track 0.00 -> 504.2 mm, vias 0 -> 2
- net COL9: track 0.00 -> 479.7 mm
- net COL2: track 0.00 -> 474.3 mm, vias 0 -> 2
- net COL0: track 0.00 -> 470.7 mm
- net COL1: track 0.00 -> 423.9 mm
- net COL10: track 0.00 -> 408.0 mm, vias 0 -> 1
- net COL11: track 0.00 -> 324.0 mm, vias 0 -> 2
- net COL12: track 0.00 -> 264.2 mm, vias 0 -> 1
- net COL14: track 0.00 -> 205.1 mm
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Other:
- outline, holes or cut-outs redrawn
