File: Voyager87.sch (KiCad schematic (older format))
At the start: 22 parts, among them J1 AVR-ISP-6, Q1 DSS60601MZ4-13, SW1 SW_Push, U1 AT90USB1286-AU, U2 PRTR5V0U2X, Y1 16MHz

Commit message: Progress
Parts:
- C5: value 10uF -> 1uF
Connections:
- net COL15: now also U1.32 (PD7); no longer U1.36 (PC1)
- net COL16: now also U1.31 (PD6); no longer U1.35 (PC0)
- net ROW0: now also U1.37 (PC2); no longer U1.32 (PD7)
