File: KBD8X-MK2.sch (KiCad schematic (older format))
At the start: 22 parts, among them J1 AVR-ISP-6, Q1 DSS60601MZ4-13, SW1 SW_Push, U1 AT90USB1286-AU, U2 PRTR5V0U2X, Y1 16MHz

Commit message: Working copy
Parts:
- removed U1: AT90USB1286-AU, Housings_DFN_QFN:QFN-64-1EP_9x9mm_Pitch0.5mm, symbol MCU_Microchip_AVR:AT90USB1286-MU
- added U1: ATmega32U4-MU, locallib:QFN-44-1EP_7x7mm_Pitch0.5mm, symbol MCU_Microchip_ATmega:ATmega32U4-MU
- C2, C3, C4, C6, C7, C8: footprint Capacitors_SMD:C_0603 -> locallib:C_0603
- C5: value 1uF -> 10uF; footprint Capacitors_SMD:C_0603 -> locallib:C_0603
- F1: footprint Fuse_Holders_and_Fuses:Fuse_SMD1206_Reflow -> Fuse_Holders_and_Fuses:Fuse_SMD1206_Wave
- RC1, RC2, RC3, RC4, RC5, RC6, RC7: footprint Resistors_SMD:R_0603 -> locallib:R_0603
- Y1: footprint Crystals:Crystal_SMD_3225-4pin_3.2x2.5mm -> locallib:Crystal_SMD_3225-4pin_3.2x2.5mm
Connections:
- net SCK is gone; now on net COL8: J1.3 (SCK)
- net +5V: now also U1.14 (VCC), U1.2 (UVCC), U1.24 (AVCC), U1.34 (VCC), U1.44 (AVCC), U1.7 (VBUS)
- net COL0: now also U1.41 (PF0)
- net COL1: now also U1.40 (PF1)
- net COL2: now also U1.39 (PF4)
- net COL3: now also U1.38 (PF5)
- net COL4: now also U1.37 (PF6)
- net COL5: now also U1.36 (PF7)
- net COL6: now also U1.32 (PC7)
- net COL7: now also U1.8 (PB0)
- net COL8: now also U1.9 (PB1)
- net D+: now also U1.4 (D+)
- net D-: now also U1.3 (D-)
- net GND: now also U1.15 (GND), U1.23 (GND), U1.35 (GND), U1.43 (GND), U1.45 (GND), U1.5 (UGND)
- net RESET: now also U1.13 (~RESET)
- net ROW0: now also U1.31 (PC6)
- net ROW1: now also U1.30 (PB6)
- net ROW2: now also U1.29 (PB5)
- net ROW3: now also U1.28 (PB4)
- net ROW4: now also U1.27 (PD7)
- net ROW5: now also U1.26 (PD6)
- net XTAL1: now also U1.17 (XTAL1)
- net XTAL2: now also U1.16 (XTAL2)
- net at RC5.1: now also U1.12 (PB7)
- net at RC4.1: now also U1.33 (~HWB~/PE2)
- net at C2.1: now also U1.6 (UCAP)
- net MISO renamed RGBLED
- net RGBLED: now also U1.11 (PB3)
- net MOSI renamed SLOCK_IND
- net SLOCK_IND: now also U1.10 (PB2)
- new net CAPS_IND: U1.1 (PE6)
- new net ROW10: U1.19 (PD1)
- new net ROW11: U1.18 (PD0)
- new net ROW6: U1.25 (PD4)
- new net ROW7: U1.22 (PD5)
- new net ROW8: U1.21 (PD3)
- new net ROW9: U1.20 (PD2)
Other:
- note added: "MISO"
- note added: "MOSI"
- note added: "SCK"
- moved on the sheet: C2, Q1, RC3, RC4, RC5, SW1
