File: matrix.sch (KiCad schematic (older format))
At the start: 283 parts

Commit message: Progress
Parts:
- MX_LALT2: footprint MX_Alps_Hybrid:MX-1.5U -> MX_Alps_Hybrid:MX-1.5U-FLIPPED
- MX_LGUI2: footprint MX_Alps_Hybrid:MX-1U -> MX_Alps_Hybrid:MX-1U-FLIPPED
- MX_RALT2: footprint MX_Alps_Hybrid:MX-1.5U-FLIPPED -> MX_Alps_Hybrid:MX-1.5U
- MX_RCTRL1, MX_RGUI1, MX_RMENU1: footprint MX_Alps_Hybrid:MX-1.25U -> MX_Alps_Hybrid:MX-1.25U-FLIPPED
Connections:
- net +5V: now also MX_LALT2.3 (LED), MX_LSHIFT2.3 (LED), MX_RCTRL2.3 (LED), MX_RETURN2.3 (LED), MX_RGUI2.3 (LED), MX_RSHIFT2.3 (LED), MX_\2.3 (LED)
- net COL0: now also MX_LSHIFT2.1 (COL)
- net COL1: now also MX_LGUI2.1 (COL); no longer MX_LGUI2.2 (ROW)
- net COL11: now also MX_RALT2.1 (COL); no longer MX_RALT2.2 (ROW)
- net COL12: now also MX_RGUI2.1 (COL), MX_RSHIFT2.1 (COL)
- net COL13: now also MX_RCTRL2.1 (COL), MX_RETURN2.1 (COL), MX_\2.1 (COL)
- net COL2: now also MX_LALT2.1 (COL)
- net COL6: now also MX_SP2.1 (COL); no longer MX_SP2.2 (ROW)
- net at D48.2 (A), MX_\1.2 (ROW): now also MX_\2.2 (ROW)
- net at MX_\1.4 (LEDGND), R48.1: now also MX_\2.4 (LEDGND)
- net at D67.2 (A), MX_LSHIFT1.2 (ROW): now also MX_LSHIFT2.2 (ROW)
- net at MX_LSHIFT1.4 (LEDGND), R67.1: now also MX_LSHIFT2.4 (LEDGND)
- net at D78.2 (A), MX_RSHIFT1.2 (ROW): now also MX_RSHIFT2.2 (ROW)
- net at MX_RSHIFT1.4 (LEDGND), R78.1: now also MX_RSHIFT2.4 (LEDGND)
- net at D85.2 (A), MX_LGUI1.2 (ROW): now also MX_LGUI2.2 (ROW); no longer MX_LGUI2.1 (COL)
- net at D86.2 (A), MX_LALT1.2 (ROW): now also MX_LALT2.2 (ROW)
- net at MX_LALT1.4 (LEDGND), R86.1: now also MX_LALT2.4 (LEDGND)
- net at D87.2 (A), MX_SP1.2 (ROW): now also MX_SP2.2 (ROW); no longer MX_SP2.1 (COL)
- net at D91.2 (A), MX_RGUI1.2 (ROW): now also MX_RALT2.2 (ROW); no longer MX_RALT2.1 (COL)
- net at D81.2 (A), MX_RMENU1.2 (ROW): now also MX_RGUI2.2 (ROW)
- net at MX_RMENU1.4 (LEDGND), R81.1: now also MX_RGUI2.4 (LEDGND)
- net at D82.2 (A), MX_RCTRL1.2 (ROW): now also MX_RCTRL2.2 (ROW)
- net at MX_RCTRL1.4 (LEDGND), R82.1: now also MX_RCTRL2.4 (LEDGND)
- net at D65.2 (A), MX_RETURN1.2 (ROW): now also MX_RETURN2.2 (ROW)
- net at MX_RETURN1.4 (LEDGND), R65.1: now also MX_RETURN2.4 (LEDGND)

Commit message: Working copy
Parts:
- added SW2, SW3: SW_SPDT, Buttons_Switches_SMD:SW_SPDT_PCM12, symbol Switch:SW_SPDT
- D1, D10, D100, D101, D108, D11, D111, D112, D113, D12, D13, D14, D17, D18, D19, D2, D20, D21, D22, D23, D24, D25, D26, D27, D28, D29, D3, D30, D31, D35, D36, D37, D38, D39, D4, D40, D41, D42, D43, D44, D45, D46, D47, D48, D5, D52, D53, D54, D55, D56, D57, D58, D59, D6, D60, D61, D62, D63, D65, D66, D67, D68, D69, D7, D70, D71, D72, D73, D74, D75, D76, D77, D78, D8, D81, D82, D84, D85, D86, D87, D9, D90, D91, D92, D93, D94, D95, D96, D97, D99: footprint Diodes_SMD:D_SOD-123 -> locallib:D_SOD-123
- MX_#0_1, MX_#1, MX_#2, MX_#3, MX_#4, MX_#5, MX_#6, MX_#7, MX_#8, MX_#9, MX_'1, MX_,1, MX_-1, MX_.1, MX_/1, MX_;1, MX_=1, MX_A1, MX_B1, MX_BACK2, MX_BACK3, MX_C1, MX_D1, MX_DEL1, MX_DN1, MX_E1, MX_END1, MX_ESC1, MX_F1, MX_FN1, MX_FN10, MX_FN11, MX_FN12, MX_FN2, MX_FN3, MX_FN4, MX_FN5, MX_FN6, MX_FN7, MX_FN8, MX_FN9, MX_G1, MX_H1, MX_HOME1, MX_I1, MX_INS1, MX_J1, MX_K1, MX_L1, MX_LFT1, MX_LSHIFT3, MX_M1, MX_N1, MX_O1, MX_P1, MX_PAUSE1, MX_PGDN1, MX_PGUP1, MX_PRINT1, MX_Q1, MX_R1, MX_RGUI2, MX_RSHIFT3, MX_RT1, MX_S1, MX_SLOCK1, MX_T1, MX_U1, MX_UP1, MX_V1, MX_W1, MX_X1, MX_Y1, MX_Z1, MX_[1, MX_\2, MX_]1, MX_`1: footprint MX_Alps_Hybrid:MX-1U -> MX_Alps_Hybrid:MXOnly-1U
- MX_BACK1: footprint MX_Alps_Hybrid:MX-2U -> MX_Alps_Hybrid:MXOnly-2U
- MX_CLOCK1, MX_RSHIFT2: footprint MX_Alps_Hybrid:MX-1.75U -> MX_Alps_Hybrid:MXOnly-1.75U
- MX_CLOCK2, MX_RCTRL1, MX_RGUI1, MX_RMENU1: footprint MX_Alps_Hybrid:MX-1.25U-FLIPPED -> MX_Alps_Hybrid:MXOnly-1.25U-FLIPPED
- MX_LALT1, MX_LCTRL1, MX_LGUI1, MX_LSHIFT2, MX_RALT1: footprint MX_Alps_Hybrid:MX-1.25U -> MX_Alps_Hybrid:MXOnly-1.25U
- MX_LALT2, MX_LCTRL2: footprint MX_Alps_Hybrid:MX-1.5U-FLIPPED -> MX_Alps_Hybrid:MXOnly-1.5U-FLIPPED
- MX_LGUI2: footprint MX_Alps_Hybrid:MX-1U-FLIPPED -> MX_Alps_Hybrid:MXOnly-1U-FLIPPED
- MX_LSHIFT1, MX_RETURN1: footprint MX_Alps_Hybrid:MX-2.25U -> MX_Alps_Hybrid:MXOnly-2.25U
- MX_RALT2, MX_RCTRL2, MX_TAB1, MX_\1: footprint MX_Alps_Hybrid:MX-1.5U -> MX_Alps_Hybrid:MXOnly-1.5U
- MX_RETURN2: footprint MX_Alps_Hybrid:MX-ISO-ReversedStabilizers -> MX_Alps_Hybrid:MXOnly-ISO-ROTATED-ReversedStabilizers
- MX_RSHIFT1: footprint MX_Alps_Hybrid:MX-2.75U -> MX_Alps_Hybrid:MXOnly-2.75U
- MX_SP1: footprint MX_Alps_Hybrid:MX-6.25U-ReversedStabilizers -> MX_Alps_Hybrid:MXOnly-6.25U-ReversedStabilizers
- MX_SP2: footprint MX_Alps_Hybrid:MX-7U-ReversedStabilizers -> MX_Alps_Hybrid:MXOnly-7U-ReversedStabilizers
- R1, R10, R100, R101, R108, R11, R111, R112, R113, R12, R13, R14, R16, R17, R18, R19, R2, R20, R21, R22, R23, R24, R25, R26, R27, R28, R29, R3, R30, R31, R32, R33, R35, R36, R37, R38, R39, R4, R40, R41, R42, R43, R44, R45, R46, R47, R48, R5, R52, R53, R54, R55, R56, R57, R58, R59, R6, R60, R61, R62, R63, R65, R66, R67, R68, R69, R7, R70, R71, R72, R73, R74, R75, R76, R77, R78, R8, R81, R82, R84, R85, R86, R87, R9, R90, R91, R95, R96, R97, R99: footprint Resistors_SMD:R_0603 -> locallib:R_0603
Connections:
- net COL10 is gone; now on net COL5: MX_#0_1.1 (COL), MX_.1.1 (COL), MX_;1.1 (COL), MX_FN9.1 (COL), MX_P1.1 (COL), MX_RALT1.1 (COL)
- net COL11 is gone; now on net COL5: MX_'1.1 (COL), MX_-1.1 (COL), MX_/1.1 (COL), MX_FN10.1 (COL), MX_RALT2.1 (COL), MX_RGUI1.1 (COL), MX_[1.1 (COL)
- net COL12 is gone; now on net COL6: MX_=1.1 (COL), MX_BACK3.1 (COL), MX_FN11.1 (COL), MX_RGUI2.1 (COL), MX_RMENU1.1 (COL), MX_RSHIFT1.1 (COL), MX_RSHIFT2.1 (COL), MX_]1.1 (COL)
- net COL13 is gone; now on net COL6: MX_BACK1.1 (COL), MX_BACK2.1 (COL), MX_FN12.1 (COL), MX_RCTRL1.1 (COL), MX_RCTRL2.1 (COL), MX_RETURN1.1 (COL), MX_RETURN2.1 (COL), MX_RSHIFT3.1 (COL), MX_\1.1 (COL), MX_\2.1 (COL)
- net COL14 is gone; now on net COL7: MX_DEL1.1 (COL), MX_INS1.1 (COL), MX_LFT1.1 (COL), MX_PRINT1.1 (COL)
- net COL15 is gone; now on net COL7: MX_DN1.1 (COL), MX_END1.1 (COL), MX_HOME1.1 (COL), MX_SLOCK1.1 (COL), MX_UP1.1 (COL)
- net COL16 is gone; now on net COL8: MX_PAUSE1.1 (COL), MX_PGDN1.1 (COL), MX_PGUP1.1 (COL), MX_RT1.1 (COL)
- net COL9 is gone; now on net COL4: MX_#9.1 (COL), MX_,1.1 (COL), MX_FN8.1 (COL), MX_L1.1 (COL), MX_O1.1 (COL)
- net COL0: now also MX_#1.1 (COL), MX_A1.1 (COL), MX_LGUI1.1 (COL), MX_LGUI2.1 (COL), MX_LSHIFT3.1 (COL), MX_Q1.1 (COL)
- net COL1: now also MX_#2.1 (COL), MX_#3.1 (COL), MX_D1.1 (COL), MX_E1.1 (COL), MX_FN1.1 (COL), MX_FN2.1 (COL), MX_LALT1.1 (COL), MX_LALT2.1 (COL), MX_S1.1 (COL), MX_W1.1 (COL), MX_X1.1 (COL), MX_Z1.1 (COL); no longer MX_#1.1 (COL), MX_A1.1 (COL), MX_LGUI1.1 (COL), MX_LGUI2.1 (COL), MX_LSHIFT3.1 (COL), MX_Q1.1 (COL)
- net COL2: now also MX_#4.1 (COL), MX_#5.1 (COL), MX_C1.1 (COL), MX_F1.1 (COL), MX_FN3.1 (COL), MX_FN4.1 (COL), MX_G1.1 (COL), MX_R1.1 (COL), MX_T1.1 (COL), MX_V1.1 (COL); no longer MX_#2.1 (COL), MX_FN1.1 (COL), MX_LALT1.1 (COL), MX_LALT2.1 (COL), MX_S1.1 (COL), MX_W1.1 (COL), MX_Z1.1 (COL)
- net COL3: now also MX_#6.1 (COL), MX_#7.1 (COL), MX_B1.1 (COL), MX_FN5.1 (COL), MX_FN6.1 (COL), MX_H1.1 (COL), MX_J1.1 (COL), MX_N1.1 (COL), MX_SP1.1 (COL), MX_SP2.1 (COL), MX_U1.1 (COL), MX_Y1.1 (COL); no longer MX_#3.1 (COL), MX_D1.1 (COL), MX_E1.1 (COL), MX_FN2.1 (COL), MX_X1.1 (COL)
- net COL4: now also MX_#8.1 (COL), MX_FN7.1 (COL), MX_I1.1 (COL), MX_K1.1 (COL), MX_M1.1 (COL); no longer MX_#4.1 (COL), MX_C1.1 (COL), MX_F1.1 (COL), MX_FN3.1 (COL), MX_R1.1 (COL)
- net COL5: no longer MX_#5.1 (COL), MX_FN4.1 (COL), MX_G1.1 (COL), MX_T1.1 (COL), MX_V1.1 (COL)
- net COL6: no longer MX_#6.1 (COL), MX_B1.1 (COL), MX_FN5.1 (COL), MX_H1.1 (COL), MX_SP1.1 (COL), MX_SP2.1 (COL), MX_Y1.1 (COL)
- net COL7: no longer MX_#7.1 (COL), MX_FN6.1 (COL), MX_J1.1 (COL), MX_N1.1 (COL), MX_U1.1 (COL)
- net COL8: no longer MX_#8.1 (COL), MX_FN7.1 (COL), MX_I1.1 (COL), MX_K1.1 (COL), MX_M1.1 (COL)
- net LEDGND: now also SW2.1 (A), SW3.1 (A); no longer R32.2, R52.2
- net ROW0: no longer D11.1 (K), D13.1 (K), D3.1 (K), D5.1 (K), D7.1 (K), D9.1 (K), D93.1 (K)
- net ROW1: now also D11.1 (K), D13.1 (K), D3.1 (K), D5.1 (K), D7.1 (K), D9.1 (K), D93.1 (K); no longer D17.1 (K), D18.1 (K), D19.1 (K), D20.1 (K), D21.1 (K), D22.1 (K), D23.1 (K), D24.1 (K), D25.1 (K), D26.1 (K), D27.1 (K), D28.1 (K), D29.1 (K), D30.1 (K), D95.1 (K), D96.1 (K), D97.1 (K)
- net ROW2: now also D17.1 (K), D19.1 (K), D21.1 (K), D23.1 (K), D25.1 (K), D27.1 (K), D29.1 (K), D95.1 (K), D97.1 (K); no longer D100.1 (K), D101.1 (K), D35.1 (K), D36.1 (K), D37.1 (K), D38.1 (K), D39.1 (K), D40.1 (K), D41.1 (K), D42.1 (K), D43.1 (K), D44.1 (K), D45.1 (K), D46.1 (K), D47.1 (K), D48.1 (K), D99.1 (K)
- net ROW3: now also D18.1 (K), D20.1 (K), D22.1 (K), D24.1 (K), D26.1 (K), D28.1 (K), D30.1 (K), D96.1 (K); no longer D31.1 (K), D52.1 (K), D53.1 (K), D54.1 (K), D55.1 (K), D56.1 (K), D57.1 (K), D58.1 (K), D59.1 (K), D60.1 (K), D61.1 (K), D62.1 (K), D63.1 (K), D65.1 (K)
- net ROW4: now also D101.1 (K), D35.1 (K), D37.1 (K), D39.1 (K), D41.1 (K), D43.1 (K), D45.1 (K), D47.1 (K), D99.1 (K); no longer D108.1 (K), D14.1 (K), D66.1 (K), D67.1 (K), D68.1 (K), D69.1 (K), D70.1 (K), D71.1 (K), D72.1 (K), D73.1 (K), D74.1 (K), D75.1 (K), D76.1 (K), D77.1 (K), D78.1 (K)
- net ROW5: now also D100.1 (K), D36.1 (K), D38.1 (K), D40.1 (K), D42.1 (K), D44.1 (K), D46.1 (K), D48.1 (K); no longer D111.1 (K), D112.1 (K), D113.1 (K), D81.1 (K), D82.1 (K), D84.1 (K), D85.1 (K), D86.1 (K), D87.1 (K), D90.1 (K), D91.1 (K)
- net CAPS_LEDGND: now reaches MX_CLOCK1.4 (LEDGND), MX_CLOCK2.4 (LEDGND), R52.1
- net at R32.1: now also SW2.2 (B); no longer MX_SLOCK1.4 (LEDGND)
- new net: R52.2, SW3.2 (B)
- new net CAPS_IND: SW3.3 (C)
- new net ROW10: D111.1 (K), D113.1 (K), D81.1 (K), D84.1 (K), D86.1 (K), D87.1 (K), D90.1 (K)
- new net ROW11: D112.1 (K), D82.1 (K), D85.1 (K), D91.1 (K)
- new net ROW6: D31.1 (K), D52.1 (K), D54.1 (K), D56.1 (K), D58.1 (K), D60.1 (K), D62.1 (K)
- new net ROW7: D53.1 (K), D55.1 (K), D57.1 (K), D59.1 (K), D61.1 (K), D63.1 (K), D65.1 (K)
- new net ROW8: D67.1 (K), D68.1 (K), D70.1 (K), D72.1 (K), D74.1 (K), D76.1 (K), D78.1 (K)
- new net ROW9: D108.1 (K), D14.1 (K), D66.1 (K), D69.1 (K), D71.1 (K), D73.1 (K), D75.1 (K), D77.1 (K)
- new net SLOCK_IND: SW2.3 (C)
- new net SLOCK_LEDGND: MX_SLOCK1.4 (LEDGND), R32.2
Other:
- moved on the sheet: R32, R52
